Commit message: fix: Resolve Gazebo Harmonic timestamp synchronization issues
This commit fixes the "jump back in time" errors and RViz resets that occurred
when running the simulation with ROS2 Jazzy and Gazebo Harmonic. The root cause
was out-of-order timestamps from Gazebo's TF and joint_states bridges.

Key changes:
- Use wall clock time (use_sim_time=False) for all TF publishers to avoid
  timestamp conflicts with Gazebo simulation time
- Add odom_to_tf node that converts /odom to TF with consistent timestamps
- Disable Gazebo's publish_odom_tf and JointStatePublisher plugins
- Remove /tf and /joint_states from ros_gz_bridge configuration
- Create energia_rover_v2.urdf.xacro with all sensors in a single file
- Archive old URDF files and unused launch files

New helper nodes added to energia_bridge:
- odom_to_tf: Broadcasts odom->base_footprint transform from odometry
- static_joint_publisher: Publishes zero joint states for continuous joints
- timestamp_republisher: Republishes sensor data with wall clock timestamps
- goal_pose_bridge: Bridges Nav2 goal poses to waypoint navigator

🤖 Generated with [Claude Code](https://claude.com/claude-code)

Co-Authored-By: Claude Opus 4.5 <noreply@anthropic.com>

File: ros2_ws/src/energia_sim/urdf/archive/sensors/lidar_camera_gps.xacro (robot description, xacro)
@@ -132,12 +132,13 @@
     <origin xyz="${ebox_length/2 - gps_radius} -0.08 ${ebox_height/2 - gps_height/2 - 0.01}" rpy="0 0 0"/>
   </joint>
-  <!-- ==================== Gazebo Plugins ==================== -->
-  <!-- RP-LIDAR A1 Plugin -->
+  <!-- ==================== Gazebo Harmonic Sensor Plugins ==================== -->
+  <!-- RP-LIDAR A1 Plugin (Gazebo Harmonic) -->
   <gazebo reference="rplidar_link">
-    <sensor name="rplidar_a1" type="ray">
+    <sensor name="rplidar_a1" type="gpu_lidar">
       <always_on>true</always_on>
       <update_rate>10</update_rate>
       <visualize>true</visualize>
-      <ray>
+      <topic>/scan</topic>
+      <lidar>
         <scan>
           <horizontal>
@@ -147,8 +148,14 @@
             <max_angle>${2*pi}</max_angle>
           </horizontal>
+          <vertical>
+            <samples>1</samples>
+            <resolution>1</resolution>
+            <min_angle>0</min_angle>
+            <max_angle>0</max_angle>
+          </vertical>
         </scan>
         <range>
-          <min>0.15</min> <!-- 15cm minimum -->
-          <max>12.0</max> <!-- 12m maximum -->
+          <min>0.15</min>
+          <max>12.0</max>
           <resolution>0.01</resolution>
         </range>
@@ -158,17 +165,13 @@
           <stddev>0.01</stddev>
         </noise>
-      </ray>
-      <plugin name="rplidar_controller" filename="libgazebo_ros_ray_sensor.so">
-        <ros>
-          <namespace>/</namespace>
-          <remapping>~/out:=scan</remapping>
-        </ros>
-        <output_type>sensor_msgs/LaserScan</output_type>
-        <frame_name>rplidar_link</frame_name>
-      </plugin>
+      </lidar>
+      <gz_frame_id>rplidar_link</gz_frame_id>
     </sensor>
-    <material>Gazebo/Black</material>
+    <material>
+      <ambient>0.1 0.1 0.1 1</ambient>
+      <diffuse>0.1 0.1 0.1 1</diffuse>
+    </material>
   </gazebo>
-  <!-- Camera Plugin (Logitech C920X) -->
+  <!-- Camera Plugin (Logitech C920X) - Gazebo Harmonic -->
   <gazebo reference="camera_link">
     <sensor name="camera" type="camera">
@@ -176,9 +179,10 @@
       <update_rate>30</update_rate>
       <visualize>true</visualize>
+      <topic>/camera/image_raw</topic>
       <camera name="camera">
-        <horizontal_fov>1.085595</horizontal_fov> <!-- ~62 degrees -->
+        <horizontal_fov>1.085595</horizontal_fov>
         <image>
-          <width>1920</width>
-          <height>1080</height>
+          <width>640</width>
+          <height>480</height>
           <format>R8G8B8</format>
         </image>
@@ -193,26 +197,23 @@
         </noise>
       </camera>
-      <plugin name="camera_controller" filename="libgazebo_ros_camera.so">
-        <ros>
-          <namespace>/</namespace>
-        </ros>
-        <camera_name>camera</camera_name>
-        <frame_name>camera_optical_link</frame_name>
-        <hack_baseline>0.0</hack_baseline>
-      </plugin>
+      <gz_frame_id>camera_optical_link</gz_frame_id>
     </sensor>
-    <material>Gazebo/DarkGrey</material>
+    <material>
+      <ambient>0.3 0.3 0.3 1</ambient>
+      <diffuse>0.3 0.3 0.3 1</diffuse>
+    </material>
   </gazebo>
-  <!-- GPS Plugin (HERE 3+) -->
+  <!-- GPS Plugin (HERE 3+) - Gazebo Harmonic NavSat -->
   <gazebo reference="gps_link">
-    <sensor name="gps_sensor" type="gps">
+    <sensor name="gps_sensor" type="navsat">
       <always_on>true</always_on>
       <update_rate>10</update_rate>
-      <gps>
+      <topic>/gps/fix</topic>
+      <navsat>
         <position_sensing>
           <horizontal>
             <noise type="gaussian">
               <mean>0.0</mean>
-              <stddev>0.005</stddev> <!-- 5mm accuracy (RTK) -->
+              <stddev>0.005</stddev>
             </noise>
           </horizontal>
@@ -220,5 +221,5 @@
             <noise type="gaussian">
               <mean>0.0</mean>
-              <stddev>0.01</stddev> <!-- 10mm vertical accuracy -->
+              <stddev>0.01</stddev>
             </noise>
           </vertical>
@@ -238,14 +239,62 @@
           </vertical>
         </velocity_sensing>
-      </gps>
-      <plugin name="gps_controller" filename="libgazebo_ros_gps_sensor.so">
-        <ros>
-          <namespace>/</namespace>
-          <remapping>~/out:=gps/fix</remapping>
-        </ros>
-        <frame_name>gps_link</frame_name>
-      </plugin>
+      </navsat>
+      <gz_frame_id>gps_link</gz_frame_id>
     </sensor>
-    <material>Gazebo/Black</material>
+    <material>
+      <ambient>0.1 0.1 0.1 1</ambient>
+      <diffuse>0.1 0.1 0.1 1</diffuse>
+    </material>
+  </gazebo>
+  <!-- IMU Sensor (commonly needed for navigation) - Gazebo Harmonic -->
+  <gazebo reference="base_link">
+    <sensor name="imu_sensor" type="imu">
+      <always_on>true</always_on>
+      <update_rate>100</update_rate>
+      <topic>/imu</topic>
+      <imu>
+        <angular_velocity>
+          <x>
+            <noise type="gaussian">
+              <mean>0.0</mean>
+              <stddev>0.0002</stddev>
+            </noise>
+          </x>
+          <y>
+            <noise type="gaussian">
+              <mean>0.0</mean>
+              <stddev>0.0002</stddev>
+            </noise>
+          </y>
+          <z>
+            <noise type="gaussian">
+              <mean>0.0</mean>
+              <stddev>0.0002</stddev>
+            </noise>
+          </z>
+        </angular_velocity>
+        <linear_acceleration>
+          <x>
+            <noise type="gaussian">
+              <mean>0.0</mean>
+              <stddev>0.017</stddev>
+            </noise>
+          </x>
+          <y>
+            <noise type="gaussian">
+              <mean>0.0</mean>
+              <stddev>0.017</stddev>
+            </noise>
+          </y>
+          <z>
+            <noise type="gaussian">
+              <mean>0.0</mean>
+              <stddev>0.017</stddev>
+            </noise>
+          </z>
+        </linear_acceleration>
+      </imu>
+      <gz_frame_id>base_link</gz_frame_id>
+    </sensor>
   </gazebo>
 </robot>

File: ros2_ws/src/energia_sim/urdf/archive/sensors/ultrasonic_sensors.xacro (robot description, xacro)
@@ -6,5 +6,5 @@
   <xacro:property name="ultrasonic_min_range" value="0.20"/> <!-- 20cm minimum -->
   <xacro:property name="ultrasonic_max_range" value="6.0"/> <!-- 600cm maximum -->
-  <xacro:property name="ultrasonic_fov" value="1.22"/> <!-- 70° cone = 1.22 radians -->
+  <xacro:property name="ultrasonic_fov" value="1.22"/> <!-- 70 deg cone = 1.22 radians -->
   <xacro:property name="ultrasonic_update_rate" value="20"/> <!-- 20 Hz -->
   <!-- ==================== Ultrasonic Sensor Macro ==================== -->
@@ -42,13 +42,14 @@
       <origin xyz="${x} ${y} ${z}" rpy="0 0 ${yaw}"/>
     </joint>
-    <!-- Gazebo sensor plugin -->
+    <!-- Gazebo Harmonic sensor plugin -->
     <gazebo reference="${name}_link">
-      <sensor name="${name}" type="ray">
+      <sensor name="${name}" type="gpu_lidar">
         <always_on>true</always_on>
         <update_rate>${ultrasonic_update_rate}</update_rate>
         <visualize>false</visualize>
-        <ray>
+        <topic>ultrasonic/${name}</topic>
+        <lidar>
           <scan>
-            <!-- Simulate 70° cone with 5 horizontal rays -->
+            <!-- Simulate 70 deg cone with 5 horizontal rays -->
             <horizontal>
               <samples>5</samples>
@@ -68,39 +69,25 @@
             <min>${ultrasonic_min_range}</min>
             <max>${ultrasonic_max_range}</max>
-            <resolution>0.01</resolution> <!-- 1cm resolution -->
+            <resolution>0.01</resolution>
           </range>
           <noise>
             <type>gaussian</type>
             <mean>0.0</mean>
-            <stddev>0.01</stddev> <!-- ±1cm accuracy -->
+            <stddev>0.01</stddev>
           </noise>
-        </ray>
-        <plugin name="${name}_controller" filename="libgazebo_ros_ray_sensor.so">
-          <ros>
-            <namespace>/ultrasonic</namespace>
-            <remapping>~/out:=${name}</remapping>
-          </ros>
-          <output_type>sensor_msgs/Range</output_type>
-          <frame_name>${name}_link</frame_name>
-          <radiation_type>ultrasound</radiation_type>
-        </plugin>
+        </lidar>
+        <gz_frame_id>${name}_link</gz_frame_id>
       </sensor>
-      <material>Gazebo/Grey</material>
+      <material>
+        <ambient>0.3 0.3 0.3 1</ambient>
+        <diffuse>0.5 0.5 0.5 1</diffuse>
+      </material>
     </gazebo>
   </xacro:macro>
   <!-- ==================== 6-Sensor Array Instantiation ==================== -->
-  <!--
-    Sensor Layout (Top-Down View):
-                        FRONT
-          [Corner L] [Front] [Corner R]
-              45°      0°       45°
-               \       |       /
-                \      |      /
-      [Side L]   \     |     /    [Side R]
-       90°        \    |    /       90°
-                   └───┴───┘
-                      |
-                    [Rear]
-                     180°
+  <!-- Sensor Layout (Top-Down View):
+       FRONT: Corner Left (45deg), Front (0deg), Corner Right (45deg)
+       SIDES: Side Left (90deg), Side Right (90deg)
+       REAR: Rear (180deg)
   -->
   <!-- Mounting heights: All sensors at 11 inches (0.2794m) from ground -->
@@ -112,5 +99,5 @@
   <xacro:property name="rear_x" value="${-chassis_length/2}"/> <!-- Rear edge -->
   <xacro:property name="side_y" value="${chassis_width/2}"/> <!-- Side edges -->
-  <!-- Front Sensor (0° - straight ahead) -->
+  <!-- Front Sensor (0 deg - straight ahead) -->
   <xacro:ultrasonic_sensor
     name="front"
@@ -120,5 +107,5 @@
     z="${sensor_z_offset}"
     yaw="0"/>
-  <!-- Corner Left Sensor (45° outward-left from front) -->
+  <!-- Corner Left Sensor (45 deg outward-left from front) -->
   <xacro:ultrasonic_sensor
     name="corner_left"
@@ -128,5 +115,5 @@
     z="${sensor_z_offset}"
     yaw="${pi/4}"/>
-  <!-- Corner Right Sensor (45° outward-right from front) -->
+  <!-- Corner Right Sensor (45 deg outward-right from front) -->
   <xacro:ultrasonic_sensor
     name="corner_right"
@@ -136,5 +123,5 @@
     z="${sensor_z_offset}"
     yaw="${-pi/4}"/>
-  <!-- Side Left Sensor (90° perpendicular left) -->
+  <!-- Side Left Sensor (90 deg perpendicular left) -->
   <!-- Positioned 9 inches back from front edge: chassis_length/2 - 9" = 13.5" - 9" = 4.5" = 0.1143m -->
   <xacro:ultrasonic_sensor
@@ -145,5 +132,5 @@
     z="${sensor_z_offset}"
     yaw="${pi/2}"/>
-  <!-- Side Right Sensor (90° perpendicular right) -->
+  <!-- Side Right Sensor (90 deg perpendicular right) -->
   <!-- Positioned 9 inches back from front edge: chassis_length/2 - 9" = 13.5" - 9" = 4.5" = 0.1143m -->
   <xacro:ultrasonic_sensor
@@ -154,5 +141,5 @@
     z="${sensor_z_offset}"
     yaw="${-pi/2}"/>
-  <!-- Rear Sensor (180° straight back) -->
+  <!-- Rear Sensor (180 deg straight back) -->
   <xacro:ultrasonic_sensor
     name="rear"
